File: rk-clock.kicad_pcb (KiCad board)
At the start: 2 copper layers, 105.4 x 106.7 mm, 102 parts, among them J1 min_display, J10 colon_control, J2 min_control, J3 tenmin_control, J4 tenmin_display, J5 hour_control, J6 tenhour_control, J7 hour_display, J8 tenhour_display, J9 colon_display, SW1 mode, SW2 increase, U1 74'4060, U10 '08, U11 '158, U12 '04, U13 '08, U14 LED-7Seg-18DIP, U15 74'4511, U16 74'163, U17 74'163, U18 '08, U19 '11, U2 74'163, U20 '02, U21 '04, U22 LED-7Seg-18DIP, U23 74'4511, U24 LED-7Seg-18DIP, U25 74'4511, U26 '08, U27 '175, U3 74'163, U30 '14, U33 '10, U35 '32, U36 '32, U37 '14, U38 '32, U4 '10, U5 '10, U6 LED-7Seg-18DIP, U7 74'4511, U8 74'163, U9 74'163, Y1 32k768

Commit message: a few changes, some routing
Parts:
- removed J3: tenmin_control, Connector_PinHeader_2.54mm:PinHeader_1x07_P2.54mm_Vertical
- removed J4: tenmin_display, Connector_PinHeader_2.54mm:PinHeader_1x07_P2.54mm_Vertical
- removed J6: tenhour_control, Connector_PinHeader_2.54mm:PinHeader_1x07_P2.54mm_Vertical
- removed J8: tenhour_display, Connector_PinHeader_2.54mm:PinHeader_1x07_P2.54mm_Vertical
- added H15: MountingHole, rk-clock:button-hole, F.Cu at (29.5, 72.1)
- added H16: MountingHole, rk-clock:button-hole, F.Cu at (29.5, 82.8)
- added NT1: Net-Tie_2, Resistor_SMD:R_0805_2012Metric_Pad1.15x1.40mm_HandSolder, B.Cu at (53.0, 89.0)
- added NT2: Net-Tie_2, Resistor_SMD:R_0805_2012Metric_Pad1.15x1.40mm_HandSolder, B.Cu at (100.7, 89.2)
- C3, C4, J5, R33, R34, R35, R36, U26, U27, U33, U35, U36, U38: moved to B.Cu
- J1: footprint Connector_PinHeader_2.54mm:PinHeader_1x07_P2.54mm_Vertical -> Connector_PinHeader_2.54mm:PinHeader_1x08_P2.54mm_Vertical
- J10: footprint Connector_PinHeader_2.54mm:PinHeader_1x01_P2.54mm_Vertical -> Connector_PinHeader_2.54mm:PinHeader_1x05_P2.54mm_Vertical; moved to B.Cu
- J2: footprint Connector_PinHeader_2.54mm:PinHeader_1x07_P2.54mm_Vertical -> Connector_PinHeader_2.54mm:PinHeader_1x08_P2.54mm_Vertical; moved to B.Cu
- J9: footprint Connector_PinHeader_2.54mm:PinHeader_1x01_P2.54mm_Vertical -> Connector_PinHeader_2.54mm:PinHeader_1x05_P2.54mm_Vertical
- U1: value 74'4060 -> '4060
- U15, U23, U25, U7: value 74'4511 -> '4511
- U16, U17, U2, U3, U8, U9: value 74'163 -> '163
- U30, U37: value '14 -> '17; moved to B.Cu
- moved U16 87.2 mm to (91.4, 51.5), turned to 270 degrees
- moved U8 87.1 mm to (43.2, 51.5), turned to 270 degrees
- moved U9 86.9 mm to (55.9, 51.5), turned to 270 degrees
- moved U17 86.8 mm to (104.1, 51.4), turned to 270 degrees
- moved U11 71.3 mm to (96.1, 29.5), turned to 270 degrees
- moved U38 51.3 mm to (75.6, 53.4), turned to 180 degrees
- moved U36 13.8 mm to (101.3, -1.29)
- moved U26 13.4 mm to (86.3, -13.8)
- moved U33 13.4 mm to (76.7, -13.8)
- moved U35 13.4 mm to (81.5, -13.8)
- moved U27 8.80 mm to (108.2, 29.5), turned to 270 degrees
- moved J1 7.77 mm to (111.1, 92.7), turned to 90 degrees
- moved J2 7.77 mm to (42.5, 57.1)
- moved J7 7.40 mm to (62.9, 92.7), turned to 90 degrees
- moved J5 7.40 mm to (90.8, 57.1)
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Connections:
- J1 pad 5: /DGND -> Net-(J1-Pad5)
- J1 pad 7: /DVCC -> Net-(J1-Pad7)
- J10 pad 1: /colon_control -> GND
- J2 pad 1: /min_bit0 -> /min_bit1
- J2 pad 2: /min_bit1 -> /min_bit2
- J2 pad 3: /min_bit2 -> /min_bit3
- J2 pad 4: /min_bit3 -> /min_bit0
- J2 pad 5: GND -> /~min_blank
- J2 pad 6: /~min_blank -> /tenmin_bit1
- J2 pad 7: VCC -> /tenmin_bit2
- J5 pad 1: /hour_bit0 -> /hour_bit1
- J5 pad 2: /hour_bit1 -> /hour_bit2
- J5 pad 3: /hour_bit2 -> /hour_bit3
- J5 pad 4: /hour_bit3 -> /hour_bit0
- J5 pad 5: GND -> /~hour_blank
- J5 pad 6: /~hour_blank -> /tenhour_bit1
- J5 pad 7: VCC -> /tenhour_bit0
- J7 pad 5: /DGND -> Net-(J7-Pad5)
- J7 pad 7: /DVCC -> Net-(J7-Pad7)
- J9 pad 1: Net-(J9-Pad1) -> /DGND
- R17 pad 2: Net-(J9-Pad1) -> Net-(J9-Pad4)
- R18 pad 2: Net-(J9-Pad1) -> Net-(J9-Pad4)
- U15 pad 1: Net-(J4-Pad2) -> Net-(J1-Pad6)
- U15 pad 2: Net-(J4-Pad3) -> Net-(J1-Pad7)
- U15 pad 4: Net-(J4-Pad6) -> Net-(J1-Pad5)
- U15 pad 6: Net-(J4-Pad4) -> /DGND
- U15 pad 7: Net-(J4-Pad1) -> Net-(J1-Pad8)
- U17 pad 11: /tenhour_bit3 -> Net-(U17-Pad11)
- U17 pad 12: /tenhour_bit2 -> Net-(U17-Pad12)
- U23 pad 1: Net-(J7-Pad2) -> Net-(J7-Pad1)
- U23 pad 2: Net-(J7-Pad3) -> Net-(J7-Pad2)
- U23 pad 4: Net-(J7-Pad6) -> Net-(J7-Pad5)
- U23 pad 6: Net-(J7-Pad4) -> Net-(J7-Pad3)
- U23 pad 7: Net-(J7-Pad1) -> Net-(J7-Pad4)
- U25 pad 1: Net-(J8-Pad2) -> Net-(J7-Pad6)
- U25 pad 2: Net-(J8-Pad3) -> /DGND
- U25 pad 4: Net-(J8-Pad6) -> Net-(J7-Pad5)
- U25 pad 6: Net-(J8-Pad4) -> /DGND
- U25 pad 7: Net-(J8-Pad1) -> Net-(J7-Pad7)
- U7 pad 1: Net-(J1-Pad2) -> Net-(J1-Pad1)
- U7 pad 2: Net-(J1-Pad3) -> Net-(J1-Pad2)
- U7 pad 4: Net-(J1-Pad6) -> Net-(J1-Pad5)
- U7 pad 6: Net-(J1-Pad4) -> Net-(J1-Pad3)
- U7 pad 7: Net-(J1-Pad1) -> Net-(J1-Pad4)
- U9 pad 11: /tenmin_bit3 -> Net-(U9-Pad11)
Routing:
- net VCC: track 22.0 -> 175.1 mm
- net /DVCC: track 167.0 -> 99.6 mm
- net Net-(J7-Pad5): track 0.00 -> 31.0 mm
- net Net-(J1-Pad5): track 0.00 -> 28.4 mm
- net Net-(J9-Pad4): track 0.00 -> 17.3 mm
- net Net-(J9-Pad1): track 15.4 -> 0.00 mm
- net Net-(J4-Pad2): track 14.7 -> 0.00 mm
- net Net-(J8-Pad2): track 14.7 -> 0.00 mm
- net Net-(J4-Pad1): track 13.5 -> 0.00 mm
- net Net-(J8-Pad1): track 13.5 -> 0.00 mm
- net /hour_bit0: track 0.00 -> 13.4 mm
- net /min_bit0: track 0.00 -> 13.4 mm
- net Net-(J4-Pad3): track 12.1 -> 0.00 mm
- net Net-(J8-Pad3): track 12.1 -> 0.00 mm
- net /DGND: track 0.00 -> 11.7 mm
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- added copper zone on B.Cu, net GND
- removed copper zone on B.Cu, net (none)
Other:
- net class Power added: clearance 0.2, trace_width 0.4, via_dia 1, via_drill 0.4
